File: Hardware/LP55231_breakout.sch (EAGLE design)
At the start: 29 parts, among them J1 USER LED, J2 USER LED, J3 USER LED, J5 To micro, U1 LP55231WQFN

Commit message: Prepping for review.
BOM created, checklist scrubbed.
Parts:
- removed J5: To micro, SparkFun-Connectors:M08NO_SILK_FEMALE_PTH
- removed LED4: LED-TRICOLOR-5050NO_IC, SparkFun-LED:LED-TRICOLOR-5050NO_IC
- added J4: USER LED, SparkFun-Connectors:M04NO_SILK_ALL_ROUND
- added LED3: TRICOLOR-5050, SparkFun-LED:LED-TRICOLOR-5050NO_IC
- C2: value 1.0uF -> 0.47uf; device SparkFun-Capacitors:1.0UF-16V-10%(0603) -> SparkFun-Capacitors:CAP0603-CAP; PROD_ID (none) -> CAP-13216; SEE-ALSO (none) -> battery-babysitter
- C3: SEE-ALSO battery-babysitter -> battery bayasitter
- C4: value 0.47uf -> 1.0uF; device SparkFun-Capacitors:CAP0603-CAP -> SparkFun-Capacitors:1.0UF-16V-10%(0603); PROD_ID CAP-13216 -> (none); SEE-ALSO battery bayasitter -> (none)
- J1: value USER LED -> To micro; device SparkFun-Connectors:M04NO_SILK_ALL_ROUND -> SparkFun-Connectors:M08NO_SILK_FEMALE_PTH
- JP1: value A0 -> A1
- JP2: value A1 -> I2C-PULLUPS; device SparkFun-Passives:JUMPER-PAD-3-2OF3_NC_BY_TRACE_SMALL -> SparkFun-Passives:JUMPER-PAD-3-NC_BY_TRACE
- JP3: value I2C-PULLUPS -> A0; device SparkFun-Passives:JUMPER-PAD-3-NC_BY_TRACE -> SparkFun-Passives:JUMPER-PAD-3-2OF3_NC_BY_TRACE_SMALL
- LED1: value LED-TRICOLOR-NO-COMPLCC-6-SMD -> TRICOLOR-PLCC-6
- LED2: value LED-TRICOLOR-5050NO_IC -> TRICOLOR-5050
- LOGO1: value OSHW-LOGOS -> SFE_LOGO_FLAME.1_INCH; device SparkFun-Aesthetics:OSHW-LOGOS -> SparkFun-Aesthetics:SFE_LOGO_FLAME.1_INCH
- LOGO3: value SFE_LOGO_FLAME.1_INCH -> OSHW-LOGOS; device SparkFun-Aesthetics:SFE_LOGO_FLAME.1_INCH -> SparkFun-Aesthetics:OSHW-LOGOS
- R1, R2: value 4.7K -> 150K; device SparkFun-Resistors:4.7KOHM-1/10W-1%(0603) -> SparkFun-Resistors:150KOHM1/10W1%(0603)
- R4, R5: value 150K -> 4.7K; device SparkFun-Resistors:150KOHM1/10W1%(0603) -> SparkFun-Resistors:4.7KOHM-1/10W-1%(0603)
Connections:
- net ADDR0: now also JP3.2; no longer JP1.2
- net ADDR1: now also JP1.2; no longer JP2.2
- net B1: now also J2.4; no longer J1.4
- net B2: now also J3.4, LED3.BLU-A; no longer J2.4, LED2.BLU-A
- net B3: now also J4.4, LED2.BLU-A; no longer J3.4, LED4.BLU-A
- net EN: now also J1.5, R1.1; no longer J5.5, R5.1
- net G1: now also J2.3; no longer J1.3
- net G2: now also J3.3, LED3.GRN-A; no longer J2.3, LED2.GRN-A
- net G3: now also J4.3, LED2.GRN-A; no longer J3.3, LED4.GRN-A
- net GND: now also C4.2, J1.1, J4.2, JP3.3, R3.2; no longer C2.2, J1.2, J5.1, JP2.3, R4.2
- net INT: now also J1.6, R2.1; no longer J5.6, R3.1
- net N$1: now also LED2.BLU-C, LED2.GRN-C, LED2.RED-C; no longer LED4.BLU-C, LED4.GRN-C, LED4.RED-C
- net N$11: now also C2.1; no longer C3.1
- net N$12: now also C2.2; no longer C3.2
- net N$13: now also C3.1; no longer C4.1
- net N$14: now also C3.2; no longer C4.2
- net N$2: now also LED3.BLU-C, LED3.GRN-C, LED3.RED-C; no longer LED2.BLU-C, LED2.GRN-C, LED2.RED-C
- net N$21: now also JP2.1, R5.2; no longer JP3.1, R2.2
- net N$22: now also JP2.3, R4.2; no longer JP3.3, R1.2
- net R1: now also J2.1; no longer J1.1
- net R2: now also J3.1, LED3.RED-A; no longer J2.1, LED2.RED-A
- net R3: now also J4.1, LED2.RED-A; no longer J3.1, LED4.RED-A
- net SCL: now also J1.4, R4.1; no longer J5.4, R1.1
- net SDA: now also J1.3, R5.1; no longer J5.3, R2.1
- net TRIG: now also J1.7, R3.1; no longer J5.7, R4.1
- net VCC: now also C1.1, J1.2, JP2.2, JP3.1, R1.2, R2.2; no longer C2.1, J5.2, JP2.1, JP3.2, R3.2, R5.2
- net VOUT: now also C4.1, J1.8; no longer C1.1, J5.8
Other:
- note added: "J1, J2, J3 are header pads for PTH RGB LEDs, such as COM-09264 or COM-00105. JP4, JP5, JP6 can be used to disable onboard LEDs when external ones are added"
- note removed: "J1, J2, J3 are header pads for PTH RGB LEDs, such as COM-09264 or COM-00105"
- moved on the sheet: C1, C2, C3, C4, J2, J3, JP1, LED2, R1, R2, R3, R4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

Commit message: Fixing review issues.
-Fiducial moved from under silk.
-Swapped numbering of LED's 2 & 3.
Connections:
- net B2: now also LED2.BLU-A; no longer LED3.BLU-A
- net B3: now also LED3.BLU-A; no longer LED2.BLU-A
- net G2: now also LED2.GRN-A; no longer LED3.GRN-A
- net G3: now also LED3.GRN-A; no longer LED2.GRN-A
- net N$1: now also LED3.BLU-C, LED3.GRN-C, LED3.RED-C; no longer LED2.BLU-C, LED2.GRN-C, LED2.RED-C
- net N$2: now also LED2.BLU-C, LED2.GRN-C, LED2.RED-C; no longer LED3.BLU-C, LED3.GRN-C, LED3.RED-C
- net R2: now also LED2.RED-A; no longer LED3.RED-A
- net R3: now also LED3.RED-A; no longer LED2.RED-A
Other:
- moved on the sheet: LED2, LED3
Changed lines of the file:
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@@
 <part name="LOGO3" library="SparkFun-Aesthetics" deviceset="OSHW-LOGO" device="S"/>
 <part name="LOGO2" library="SparkFun-Aesthetics" deviceset="SFE_LOGO_NAME" device=".1_INCH"/>
-<part name="LED2" library="SparkFun-LED" deviceset="LED-TRICOLOR-5050" device="NO_IC" value="TRICOLOR-5050"/>
+<part name="LED3" library="SparkFun-LED" deviceset="LED-TRICOLOR-5050" device="NO_IC" value="TRICOLOR-5050"/>
 <part name="J2" library="SparkFun-Connectors" deviceset="M04" device="NO_SILK_ALL_ROUND" value="USER LED"/>
 <part name="J3" library="SparkFun-Connectors" deviceset="M04" device="NO_SILK_ALL_ROUND" value="USER LED"/>
@@
 <part name="GND2" library="SparkFun-Aesthetics" deviceset="GND" device=""/>
 <part name="LOGO1" library="SparkFun-Aesthetics" deviceset="SFE_LOGO_FLAME" device=".1_INCH"/>
-<part name="LED3" library="SparkFun-LED" deviceset="LED-TRICOLOR-5050" device="NO_IC" value="TRICOLOR-5050"/>
+<part name="LED2" library="SparkFun-LED" deviceset="LED-TRICOLOR-5050" device="NO_IC" value="TRICOLOR-5050"/>
 </parts>
 <sheets>
@@
 <instance part="LOGO3" gate="G$1" x="233.68" y="45.72"/>
 <instance part="LOGO2" gate="G$1" x="88.9" y="2.54"/>
-<instance part="LED2" gate="D1" x="185.42" y="76.2" rot="R180"/>
+<instance part="LED3" gate="D1" x="185.42" y="76.2" rot="R180"/>
 <instance part="J2" gate="G$1" x="187.96" y="139.7" rot="MR0"/>
 <instance part="J3" gate="G$1" x="187.96" y="99.06" rot="MR0"/>
@@
 <instance part="GND2" gate="1" x="48.26" y="106.68"/>
 <instance part="LOGO1" gate="G$1" x="78.74" y="2.54"/>
-<instance part="LED3" gate="D1" x="190.5" y="119.38" rot="R180"/>
+<instance part="LED2" gate="D1" x="190.5" y="119.38" rot="R180"/>
 </instances>
 <busses>
@@
 <pinref part="U1" gate="G$1" pin="R3/D9"/>
 <wire x1="139.7" y1="93.98" x2="162.56" y2="93.98" width="0.1524" layer="91"/>
-<pinref part="LED2" gate="D1" pin="RED-A"/>
+<pinref part="LED3" gate="D1" pin="RED-A"/>
 <wire x1="170.18" y1="78.74" x2="162.56" y2="78.74" width="0.1524" layer="91"/>
 <wire x1="162.56" y1="78.74" x2="162.56" y2="93.98" width="0.1524" layer="91"/>
@@
 <wire x1="160.02" y1="91.44" x2="139.7" y2="91.44" width="0.1524" layer="91"/>
 <wire x1="160.02" y1="91.44" x2="160.02" y2="76.2" width="0.1524" layer="91"/>
-<pinref part="LED2" gate="D1" pin="GRN-A"/>
+<pinref part="LED3" gate="D1" pin="GRN-A"/>
 <wire x1="160.02" y1="76.2" x2="170.18" y2="76.2" width="0.1524" layer="91"/>
 <pinref part="J4" gate="G$1" pin="3"/>
@@
 <pinref part="U1" gate="G$1" pin="B3/D6"/>
 <wire x1="139.7" y1="88.9" x2="157.48" y2="88.9" width="0.1524" layer="91"/>
-<pinref part="LED2" gate="D1" pin="BLU-A"/>
+<pinref part="LED3" gate="D1" pin="BLU-A"/>
 <wire x1="170.18" y1="73.66" x2="157.48" y2="73.66" width="0.1524" layer="91"/>
 <wire x1="157.48" y1="73.66" x2="157.48" y2="88.9" width="0.1524" layer="91"/>
@@
 <wire x1="182.88" y1="104.14" x2="172.72" y2="104.14" width="0.1524" layer="91"/>
 <wire x1="172.72" y1="104.14" x2="172.72" y2="116.84" width="0.1524" layer="91"/>
-<pinref part="LED3" gate="D1" pin="BLU-A"/>
+<pinref part="LED2" gate="D1" pin="BLU-A"/>
 <wire x1="172.72" y1="116.84" x2="175.26" y2="116.84" width="0.1524" layer="91"/>
 <junction x="172.72" y="104.14"/>
@@
 <junction x="167.64" y="104.14"/>
 <wire x1="167.64" y1="119.38" x2="167.64" y2="121.92" width="0.1524" layer="91"/>
-<pinref part="LED3" gate="D1" pin="RED-A"/>
+<pinref part="LED2" gate="D1" pin="RED-A"/>
 <wire x1="167.64" y1="121.92" x2="175.26" y2="121.92" width="0.1524" layer="91"/>
 </segment>
@@
 <junction x="170.18" y="101.6"/>
 <wire x1="170.18" y1="116.84" x2="170.18" y2="119.38" width="0.1524" layer="91"/>
-<pinref part="LED3" gate="D1" pin="GRN-A"/>
+<pinref part="LED2" gate="D1" pin="GRN-A"/>
 <wire x1="170.18" y1="119.38" x2="175.26" y2="119.38" width="0.1524" layer="91"/>
 </segment>
@@
 <junction x="215.9" y="76.2"/>
 <wire x1="200.66" y1="73.66" x2="215.9" y2="73.66" width="0.1524" layer="91"/>
-<pinref part="LED2" gate="D1" pin="BLU-C"/>
-<pinref part="LED2" gate="D1" pin="GRN-C"/>
-<pinref part="LED2" gate="D1" pin="RED-C"/>
+<pinref part="LED3" gate="D1" pin="BLU-C"/>
+<pinref part="LED3" gate="D1" pin="GRN-C"/>
+<pinref part="LED3" gate="D1" pin="RED-C"/>
 <pinref part="JP6" gate="G$1" pin="2"/>
 <wire x1="215.9" y1="73.66" x2="215.9" y2="71.12" width="0.1524" layer="91"/>
@@
 <wire x1="215.9" y1="116.84" x2="215.9" y2="109.22" width="0.1524" layer="91"/>
 <junction x="215.9" y="116.84"/>
-<pinref part="LED3" gate="D1" pin="BLU-C"/>
-<pinref part="LED3" gate="D1" pin="GRN-C"/>
-<pinref part="LED3" gate="D1" pin="RED-C"/>
-</segment>
-</net>
+<pinref part="LED2" gate="D1" pin="BLU-C"/>
+<pinref part="LED2" gate="D1" pin="GRN-C"/>
+<pinref part="LED2" gate="D1" pin="RED-C"/>
+</segment>
+</net>

Commit message: Updates to PCB after testing.
Preparing for second round of prototypes.
Parts:
- LED1: value TRICOLOR-PLCC-6 -> TRICOLOR-5050; device SparkFun-LED:LED-TRICOLOR-NO-COMPLCC-6-SMD -> SparkFun-LED:LED-TRICOLOR-5050NO_IC
Connections:
- net B1: now also LED1.RED-A; no longer LED1.BLU
- net G1: now also LED1.BLU-A; no longer LED1.GRN
- net N$3: now also LED1.BLU-C, LED1.GRN-C, LED1.RED-C; no longer LED1.BC, LED1.GC, LED1.RC
- net R1: now also LED1.GRN-A; no longer LED1.RED
Other:
- moved on the sheet: JP4
Changed lines of the file:
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@@
 <?xml version="1.0" encoding="utf-8"?>
 <!DOCTYPE eagle SYSTEM "eagle.dtd">
-<eagle version="7.3.0">
+<eagle version="7.5.0">
 <drawing>
 <settings>
@@
 <part name="GND7" library="SparkFun-Aesthetics" deviceset="GND" device=""/>
 <part name="SUPPLY5" library="SparkFun-Aesthetics" deviceset="VCC" device=""/>
-<part name="LED1" library="SparkFun-LED" deviceset="LED-TRICOLOR-NO-COM" device="PLCC-6-SMD" value="TRICOLOR-PLCC-6"/>
 <part name="C4" library="SparkFun-Capacitors" deviceset="1.0UF-16V-10%(0603)" device="" value="1.0uF"/>
 <part name="C1" library="SparkFun-Capacitors" deviceset="1.0UF-16V-10%(0603)" device="" value="1.0uF"/>
@@
 <part name="LOGO1" library="SparkFun-Aesthetics" deviceset="SFE_LOGO_FLAME" device=".1_INCH"/>
 <part name="LED2" library="SparkFun-LED" deviceset="LED-TRICOLOR-5050" device="NO_IC" value="TRICOLOR-5050"/>
+<part name="LED1" library="SparkFun-LED" deviceset="LED-TRICOLOR-5050" device="NO_IC" value="TRICOLOR-5050"/>
 </parts>
 <sheets>
@@
 1,0 - 0x34
 1,1 - 0x35</text>
-<text x="190.5" y="167.64" size="1.778" layer="97" font="vector">J1, J2, J3 are header
-pads for PTH RGB LEDs,
-such as COM-09264 or COM-00105.
-JP4, JP5, JP6 can be used to disable
-onboard LEDs when external ones
-are added</text>
+<text x="157.48" y="170.18" size="1.778" layer="97" font="vector">J1, J2, J3 are header pads for
+PTH RGB LEDs, such as COM-09264
+or COM-00105.  JP4, JP5, JP6 can
+be used to disable onboard LEDs
+when external ones are added</text>
 <text x="71.12" y="172.72" size="1.778" layer="97" font="vector">Disconnect JP3 to defeat
 onboard I2C pullup resistors</text>
@@
 <instance part="GND7" gate="1" x="142.24" y="68.58"/>
 <instance part="SUPPLY5" gate="G$1" x="114.3" y="134.62"/>
-<instance part="LED1" gate="G$1" x="177.8" y="162.56"/>
 <instance part="C4" gate="G$1" x="142.24" y="76.2"/>
 <instance part="C1" gate="G$1" x="99.06" y="124.46"/>
 <instance part="GND13" gate="1" x="215.9" y="55.88"/>
 <instance part="GND12" gate="1" x="215.9" y="93.98"/>
-<instance part="GND11" gate="1" x="215.9" y="142.24"/>
+<instance part="GND11" gate="1" x="215.9" y="139.7"/>
 <instance part="GND4" gate="1" x="99.06" y="116.84"/>
 <instance part="C2" gate="G$1" x="127" y="139.7" rot="R90">
@@
 <instance part="FD1" gate="G$1" x="243.84" y="17.78"/>
 <instance part="GND5" gate="1" x="104.14" y="68.58"/>
-<instance part="JP4" gate="G$1" x="215.9" y="152.4" rot="R90"/>
+<instance part="JP4" gate="G$1" x="215.9" y="149.86" rot="R90"/>
 <instance part="JP5" gate="G$1" x="215.9" y="104.14" rot="R90"/>
 <instance part="JP6" gate="G$1" x="215.9" y="66.04" rot="R90"/>
@@
 <instance part="LOGO1" gate="G$1" x="78.74" y="2.54"/>
 <instance part="LED2" gate="D1" x="190.5" y="119.38" rot="R180"/>
+<instance part="LED1" gate="D1" x="190.5" y="160.02" rot="R180"/>
 </instances>
 <busses>
@@
 <wire x1="139.7" y1="114.3" x2="160.02" y2="114.3" width="0.1524" layer="91"/>
 <wire x1="160.02" y1="114.3" x2="160.02" y2="137.16" width="0.1524" layer="91"/>
-<pinref part="LED1" gate="G$1" pin="RED"/>
-<wire x1="160.02" y1="137.16" x2="160.02" y2="162.56" width="0.1524" layer="91"/>
-<wire x1="160.02" y1="162.56" x2="165.1" y2="162.56" width="0.1524" layer="91"/>
+<wire x1="160.02" y1="137.16" x2="160.02" y2="160.02" width="0.1524" layer="91"/>
+<wire x1="160.02" y1="160.02" x2="175.26" y2="160.02" width="0.1524" layer="91"/>
 <pinref part="J2" gate="G$1" pin="1"/>
 <wire x1="182.88" y1="137.16" x2="160.02" y2="137.16" width="0.1524" layer="91"/>
 <junction x="160.02" y="137.16"/>
+<pinref part="LED1" gate="D1" pin="GRN-A"/>
 </segment>
 </net>
@@
 <wire x1="139.7" y1="111.76" x2="162.56" y2="111.76" width="0.1524" layer="91"/>
 <wire x1="162.56" y1="111.76" x2="162.56" y2="142.24" width="0.1524" layer="91"/>
-<pinref part="LED1" gate="G$1" pin="GRN"/>
-<wire x1="162.56" y1="142.24" x2="162.56" y2="160.02" width="0.1524" layer="91"/>
-<wire x1="162.56" y1="160.02" x2="165.1" y2="160.02" width="0.1524" layer="91"/>
+<wire x1="162.56" y1="142.24" x2="162.56" y2="157.48" width="0.1524" layer="91"/>
+<wire x1="162.56" y1="157.48" x2="175.26" y2="157.48" width="0.1524" layer="91"/>
 <pinref part="J2" gate="G$1" pin="3"/>
 <wire x1="182.88" y1="142.24" x2="162.56" y2="142.24" width="0.1524" layer="91"/>
 <junction x="162.56" y="142.24"/>
+<pinref part="LED1" gate="D1" pin="BLU-A"/>
 </segment>
 </net>
@@
 <wire x1="139.7" y1="109.22" x2="157.48" y2="109.22" width="0.1524" layer="91"/>
 <wire x1="157.48" y1="109.22" x2="157.48" y2="144.78" width="0.1524" layer="91"/>
-<pinref part="LED1" gate="G$1" pin="BLU"/>
-<wire x1="157.48" y1="144.78" x2="157.48" y2="165.1" width="0.1524" layer="91"/>
-<wire x1="157.48" y1="165.1" x2="165.1" y2="165.1" width="0.1524" layer="91"/>
+<wire x1="157.48" y1="144.78" x2="157.48" y2="162.56" width="0.1524" layer="91"/>
+<wire x1="157.48" y1="162.56" x2="175.26" y2="162.56" width="0.1524" layer="91"/>
 <pinref part="J2" gate="G$1" pin="4"/>
 <wire x1="182.88" y1="144.78" x2="157.48" y2="144.78" width="0.1524" layer="91"/>
 <junction x="157.48" y="144.78"/>
+<pinref part="LED1" gate="D1" pin="RED-A"/>
 </segment>
 </net>
@@
 <pinref part="GND11" gate="1" pin="GND"/>
 <pinref part="JP4" gate="G$1" pin="1"/>
-<wire x1="215.9" y1="144.78" x2="215.9" y2="147.32" width="0.1524" layer="91"/>
+<wire x1="215.9" y1="142.24" x2="215.9" y2="144.78" width="0.1524" layer="91"/>
 </segment>
 <segment>
@@
 <net name="N$3" class="0">
 <segment>
-<pinref part="LED1" gate="G$1" pin="BC"/>
+<wire x1="215.9" y1="157.48" x2="215.9" y2="160.02" width="0.1524" layer="91"/>
 <wire x1="215.9" y1="160.02" x2="215.9" y2="162.56" width="0.1524" layer="91"/>
-<wire x1="215.9" y1="162.56" x2="215.9" y2="165.1" width="0.1524" layer="91"/>
-<wire x1="215.9" y1="165.1" x2="187.96" y2="165.1" width="0.1524" layer="91"/>
-<pinref part="LED1" gate="G$1" pin="RC"/>
-<wire x1="187.96" y1="162.56" x2="215.9" y2="162.56" width="0.1524" layer="91"/>
-<junction x="215.9" y="162.56"/>
-<pinref part="LED1" gate="G$1" pin="GC"/>
-<wire x1="187.96" y1="160.02" x2="215.9" y2="160.02" width="0.1524" layer="91"/>
+<wire x1="215.9" y1="162.56" x2="205.74" y2="162.56" width="0.1524" layer="91"/>
+<junction x="215.9" y="160.02"/>
+<wire x1="205.74" y1="160.02" x2="215.9" y2="160.02" width="0.1524" layer="91"/>
 <pinref part="JP4" gate="G$1" pin="2"/>
-<wire x1="215.9" y1="160.02" x2="215.9" y2="157.48" width="0.1524" layer="91"/>
-<junction x="215.9" y="160.02"/>
-</segment>
-</net>
+<wire x1="205.74" y1="157.48" x2="215.9" y2="157.48" width="0.1524" layer="91"/>
+<wire x1="215.9" y1="157.48" x2="215.9" y2="154.94" width="0.1524" layer="91"/>
+<junction x="215.9" y="157.48"/>
+<pinref part="LED1" gate="D1" pin="BLU-C"/>
+<pinref part="LED1" gate="D1" pin="GRN-C"/>
+<pinref part="LED1" gate="D1" pin="RED-C"/>
+</segment>
+</net>

Commit message: Updates after group review.
Addressing things in issue #3:
-bump version number
-Add silk indicating flooded/empty configuration on A0/A1
-space out passives on front (check tkeepout)
-remove extra junction dot between 150k res and Vcc on schematic
Other:
- note added: "V02"
- note removed: "V01"
Changed lines of the file:
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@@
 <plain>
 <text x="170.18" y="10.16" size="2.54" layer="94" font="vector">Byron Jacquot</text>
-<text x="238.76" y="7.62" size="2.54" layer="94" font="vector">V01</text>
+<text x="238.76" y="7.62" size="2.54" layer="94" font="vector">V02</text>
 <text x="10.16" y="175.26" size="1.778" layer="97" font="vector">VCC Range from 2.7 to 5.5 VDC</text>
 <text x="33.02" y="53.34" size="1.778" layer="97" font="vector">JP1, JP2 configure
@@
 <wire x1="33.02" y1="154.94" x2="33.02" y2="160.02" width="0.1524" layer="91"/>
 <wire x1="33.02" y1="160.02" x2="38.1" y2="160.02" width="0.1524" layer="91"/>
-<junction x="40.64" y="160.02"/>
 <wire x1="38.1" y1="160.02" x2="40.64" y2="160.02" width="0.1524" layer="91"/>
 </segment>
